Commit message: robot working

File: exproblab_ass3/urdf/my_robot.urdf (robot description, URDF)
Before this commit: robot my_robot, 11 links, 10 joints
Links:
- added link camera_link, mass 1e-5; collision box size=0.05 0.05 0.05; visual box size=0.05 0.05 0.05
Joints:
- added joint camera_joint: type fixed, parent cluedo_link, child camera_link, origin xyz=0 0 0.05 rpy=0 0 0, axis 0 1 0
