Commit message: move_base che fungegit add .git add .git add .git add .git add .git add .git add .git add .git add .git add .git add .git add .

File: exproblab_ass3/urdf/my_robot_backup.urdf (robot description, URDF)
Before this commit: robot my_robot, 12 links, 11 joints
Joints:
- joint joint_left_wheel: origin xyz=-0.05 0.15 0 rpy=0 0 0 -> xyz=-0.05 -0.15 0 rpy=0 0 0
- joint joint_right_wheel: origin xyz=-0.05 -0.15 0 rpy=0 0 0 -> xyz=-0.05 0.15 0 rpy=0 0 0
